File: keyboard pcb.sch (KiCad schematic (older format))
At the start: 18 parts, among them J1 TYPE-C-31-M-17, SW1 RESET, U1 AT90USB1286-MU, U2A1 OP07, Y1 16MHz

Commit message: Schematic
Schematic mostly done, i think
Parts:
- removed J1: TYPE-C-31-M-17, SamacSys_Parts:TYPEC31M17, symbol SamacSys_Parts:TYPE-C-31-M-17
- added D1, D10, D100, D101, D102, D11, D12, D13, D14, D15, D16, D17, D18, D19, D2, D20, D21, D22, D23, D24, D25, D26, D27, D28, D29, D3, D30, D31, D32, D33, D34, D35, D36, D37, D38, D39, D4, D40, D41, D42, D43, D44, D45, D46, D47, D48, D49, D5, D50, D51, D52, D53, D54, D55, D56, D57, D58, D59, D6, D60, D61, D62, D63, D64, D65, D66, D67, D68, D69, D7, D70, D71, D72, D73, D74, D75, D76, D77, D78, D79, D8, D80, D81, D82, D83, D84, D85, D86, D87, D88, D89, D9, D90, D91, D92, D93, D94, D95, D96, D97, D98, D99: SOD-123, random-keyboard-parts:D_SOD-123-Pretty, symbol Device:D_Small
- added F1: 500mA, Fuse:Fuse_1206_3216Metric, symbol Device:Polyfuse_Small
- added J1, J2, J3, J4, J5, J6: Conn_01x08, Connector_PinHeader_1.00mm:PinHeader_1x08_P1.00mm_Vertical, symbol Connector_Generic:Conn_01x08
- added J7: USB_C_Receptacle_USB2.0, Connector_USB:USB_C_Receptacle_HRO_TYPE-C-31-M-12, symbol Connector:USB_C_Receptacle_USB2.0
- added J?: Conn_01x03, symbol Connector_Generic:Conn_01x03
- added J?: Conn_01x05, symbol Connector_Generic:Conn_01x05
- added J?: Conn_01x04, symbol Connector_Generic:Conn_01x04
- added JP1: 5, Jumper:SolderJumper-3_P1.3mm_Bridged12_Pad1.0x1.5mm_NumberLabels, symbol Jumper:SolderJumper_3_Bridged12
- added MX1, MX10, MX100, MX101, MX102, MX11, MX12, MX13, MX14, MX15, MX16, MX17, MX18, MX19, MX2, MX20, MX21, MX22, MX23, MX24, MX25, MX26, MX27, MX28, MX29, MX3, MX30, MX31, MX32, MX33, MX34, MX35, MX36, MX37, MX38, MX39, MX4, MX40, MX41, MX42, MX43, MX44, MX45, MX46, MX47, MX48, MX49, MX5, MX50, MX51, MX52, MX53, MX54, MX55, MX56, MX57, MX58, MX59, MX6, MX60, MX61, MX62, MX63, MX64, MX65, MX66, MX67, MX68, MX69, MX7, MX70, MX71, MX72, MX73, MX74, MX75, MX76, MX77, MX78, MX79, MX8, MX80, MX81, MX82, MX83, MX84, MX85, MX86, MX87, MX88, MX89, MX9, MX90, MX91, MX92, MX93, MX94, MX95, MX96, MX97, MX98, MX99: MX-NoLED, MX_Only:MXOnly-1U-Hotswap-Antishear, symbol MX_Alps_Hybrid:MX-NoLED
- added R5, R6: 5.1k, Resistor_SMD:R_0805_2012Metric, symbol Device:R_Small
- added U1: MCP1825S, Package_TO_SOT_SMD:SOT-223-3_TabPin2, symbol Regulator_Linear:MCP1825S
- renumbered C7 to C3, C3 to C4, C4 to C5, C5 to C6, C6 to C7, D1 to LED1, D2 to LED2, R4 to R1, R3 to R2, R1 to R3, R2 to R4, U1 to U2
Connections:
- net labels added: COL0, COL1, COL10, COL11, COL12, COL13, COL14, COL15, COL16, COL2, COL3, COL4, COL5, COL6, COL7, COL8, COL9, ROW0, ROW1, ROW2, ROW3, ROW4, ROW5
- wire segments 121 -> 889
- no-connect marks 0 -> 2
Other:
- moved on the sheet: C3, C4, C5, C6, C7, LED1, LED2, R1, R2, R3, R4, SW1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

Commit message: Various changes
Mostly done i think
Parts:
- removed J1, J3: Conn_01x08, Connector_PinHeader_1.00mm:PinHeader_1x08_P1.00mm_Vertical, symbol Connector_Generic:Conn_01x08
- added C8: 1uF, Capacitor_SMD:C_0603_1608Metric, symbol Device:C_Small
- added J2, J7, J9: E, Connector_PinHeader_1.00mm:PinHeader_1x02_P1.00mm_Vertical, symbol Connector_Generic:Conn_01x02
- added J3, J8: A, Connector_PinHeader_1.00mm:PinHeader_1x04_P1.00mm_Vertical, symbol Connector_Generic:Conn_01x04
- added J5: E, Connector_PinHeader_1.00mm:PinHeader_1x01_P1.00mm_Vertical, symbol Connector_Generic:Conn_01x01
- added R5, R6: 22, Resistor_SMD:R_0603_1608Metric, symbol Device:R_Small
- C1, C2, C3, C4, C5, C6, C7: footprint Capacitor_SMD:C_0805_2012Metric -> Capacitor_SMD:C_0603_1608Metric
- J1: renamed from J?; value Conn_01x03 -> RGB; footprint (none) -> Connector_PinHeader_1.00mm:PinHeader_1x03_P1.00mm_Vertical
- J10: renamed from J?; value Conn_01x04 -> OLED; footprint (none) -> Connector_PinHeader_1.00mm:PinHeader_1x04_P1.00mm_Vertical
- J11: renamed from J4; value Conn_01x08 -> F
- J12: renamed from J5; value Conn_01x08 -> B
- J13: renamed from J6; value Conn_01x08 -> D
- J4: renamed from J?; value Conn_01x05 -> Encoder; footprint (none) -> Connector_PinHeader_1.00mm:PinHeader_1x05_P1.00mm_Vertical
- J6: renamed from J2; value Conn_01x08 -> C
- R1, R2, R3, R4: footprint Resistor_SMD:R_0805_2012Metric -> Resistor_SMD:R_0603_1608Metric
- R7: renamed from R5; footprint Resistor_SMD:R_0805_2012Metric -> Resistor_SMD:R_0603_1608Metric
- R8: renamed from R6; footprint Resistor_SMD:R_0805_2012Metric -> Resistor_SMD:R_0603_1608Metric
- renumbered J7 to J14
Connections:
- net B6 is gone; now on net DRGB: J12.7 (Pin_7), U2.16 (PB6)
- net B7 is gone; now on net SW: J12.8 (Pin_8), U2.17 (PB7)
- net C0 is gone; now on net COL14: J6.1 (Pin_1), U2.35 (PC0)
- net C1 is gone; now on net COL13: J6.2 (Pin_2), U2.36 (PC1)
- net C2 is gone; now on net COL12: J6.3 (Pin_3), U2.37 (PC2)
- net C3 is gone; now on net COL11: J6.4 (Pin_4), U2.38 (PC3)
- net C4 is gone; now on net COL10: J6.5 (Pin_5), U2.39 (PC4)
- net C5 is gone; now on net COL9: J6.6 (Pin_6), U2.40 (PC5)
- net C6 is gone; now on net COL8: J6.7 (Pin_7), U2.41 (PC6)
- net C7 is gone; now on net COL7: J6.8 (Pin_8), U2.42 (PC7)
- net D0 is gone; now on net SCL: J13.1 (Pin_1), U2.25 (PD0)
- net D1 is gone; now on net SDA: J13.2 (Pin_2), U2.26 (PD1)
- net D2 is gone; now on net ROW0: J13.3 (Pin_3), U2.27 (PD2)
- net D3 is gone; now on net ROW1: J13.4 (Pin_4), U2.28 (PD3)
- net D4 is gone; now on net ROW2: J13.5 (Pin_5), U2.29 (PD4)
- net D5 is gone; now on net ROW3: J13.6 (Pin_6), U2.30 (PD5)
- net D6 is gone; now on net ROW4: J13.7 (Pin_7), U2.31 (PD6), U2A1.3 (+)
- net D7 is gone; now on net ROW5: J13.8 (Pin_8), U2.32 (PD7)
- net E0 is gone; now on net COL16: U2.33 (PE0)
- net E1 is gone; now on net COL15: U2.34 (PE1)
- net E4 is gone; now on net DT: U2.18 (PE4)
- net E5 is gone; now on net CLK: U2.19 (PE5)
- net F1 is gone; now on net COL6: J11.2 (Pin_2), U2.60 (PF1)
- net F2 is gone; now on net COL5: J11.3 (Pin_3), U2.59 (PF2)
- net F3 is gone; now on net COL4: J11.4 (Pin_4), U2.58 (PF3)
- net F4 is gone; now on net COL3: J11.5 (Pin_5), U2.57 (PF4)
- net F5 is gone; now on net COL2: J11.6 (Pin_6), U2.56 (PF5)
- net F6 is gone; now on net COL1: J11.7 (Pin_7), U2.55 (PF6)
- net F7 is gone; now on net COL0: J11.8 (Pin_8), U2.54 (PF7)
- net +5V: now also J1.3 (Pin_3), J10.2 (Pin_2), J4.2 (Pin_2), JP1.2 (C), U1.3 (VO); no longer JP1.1 (A)
- net A0: now also J3.1 (Pin_1)
- net A1: now also J3.2 (Pin_2)
- net A2: now also J3.3 (Pin_3)
- net A3: now also J3.4 (Pin_4)
- net A4: now also J8.1 (Pin_1)
- net A5: now also J8.2 (Pin_2)
- net A6: now also J8.3 (Pin_3)
- net A7: now also J8.4 (Pin_4)
- net COL11: now also MX68.1 (COL), MX69.1 (COL), MX70.1 (COL), MX71.1 (COL)
- net COL15: now also MX92.1 (COL), MX93.1 (COL), MX94.1 (COL), MX95.1 (COL), J2.1 (Pin_1)
- net COL16: now also J2.2 (Pin_2)
- net COL3: now also MX20.1 (COL), MX21.1 (COL), MX22.1 (COL), MX23.1 (COL)
- net COL7: now also MX44.1 (COL), MX45.1 (COL), MX46.1 (COL), MX47.1 (COL)
- net D+: now also R6.1; no longer J14.A6 (D+), J14.B6 (D+)
- net D-: now also R5.1; no longer J14.A7 (D-), J14.B7 (D-)
- net E2: now also J5.1 (Pin_1)
- net E6: now also J9.2 (Pin_2)
- net E7: now also J9.1 (Pin_1)
- net GND: now also J1.1 (Pin_1), J10.1 (Pin_1), J4.1 (Pin_1), C8.2
- net VBUS: now also JP1.1 (A), C8.1; no longer JP1.3 (B)
- net at C3.1, U2.7 (UCAP): now also JP1.3 (B); no longer JP1.2 (C), U1.3 (VO)
- net DRGB: now reaches J1.2 (Pin_2)
- net SW: now reaches J4.3 (Pin_3)
- net DT: now reaches J4.4 (Pin_4)
- net DT: now also J7.2 (Pin_2)
- net CLK: now reaches J4.5 (Pin_5)
- net CLK: now also J7.1 (Pin_1)
- net SCL: now reaches J10.3 (Pin_3)
- net SDA: now reaches J10.4 (Pin_4)
- new net Data1+: J14.A6 (D+), J14.B6 (D+), R6.2
- new net Data1-: J14.A7 (D-), J14.B7 (D-), R5.2
- no-connect marks 2 -> 5
Other:
- moved on the sheet: C3, J1, J10, J4, R7, R8, U1

Commit message: added values for JLCPCB
added field value for JLCPCB
Parts:
- C1, C2: LCSC (none) -> C1634
- C3, C8: LCSC (none) -> C15849
- C4, C5, C6, C7: LCSC (none) -> C14663
- D1, D10, D100, D101, D102, D11, D12, D13, D14, D15, D16, D17, D18, D19, D2, D20, D21, D22, D23, D24, D25, D26, D27, D28, D29, D3, D30, D31, D32, D33, D34, D35, D36, D37, D38, D39, D4, D40, D41, D42, D43, D44, D45, D46, D47, D48, D49, D5, D50, D51, D52, D53, D54, D55, D56, D57, D58, D59, D6, D60, D61, D62, D63, D64, D65, D66, D67, D68, D69, D7, D70, D71, D72, D73, D74, D75, D76, D77, D78, D79, D8, D80, D81, D82, D83, D84, D85, D86, D87, D88, D89, D9, D90, D91, D92, D93, D94, D95, D96, D97, D98, D99: LCSC (none) -> C81598
- F1: footprint Fuse:Fuse_1206_3216Metric -> Fuse:Fuse_0603_1608Metric; LCSC (none) -> C2757929
- J14: LCSC (none) -> C165948
- LED1: LCSC (none) -> C72041
- LED2: LCSC (none) -> C72038
- R1: LCSC (none) -> C25804
- R2, R3, R4: LCSC (none) -> C21190
- R5, R6: LCSC (none) -> C23345
- R7, R8: LCSC (none) -> C23186
- U2: LCSC (none) -> C619147
- U2A1: LCSC (none) -> C7433
- Y1: LCSC (none) -> C13738
