File: keyboard-pcb.kicad_pcb (KiCad board)
At the start: 2 copper layers, 323.9 x 145.3 mm, 244 parts, among them J1 RGB, J10 OLED, J11 F, J12 B, J13 D, J14 USB_C_Receptacle_USB2.0, J2 E, J3 A, J4 Encoder, J5 E, J6 C, J7 E, J8 A, J9 E, SW1 RESET, U1 MCP1825S, U2 AT90USB1286-MU, U2A1 OP07, Y1 16MHz

Commit message: fixes and 3d
fixed libraries and added 3d models
Parts:
- removed G***: LOGO, Logo:poto

Commit message: finished?
rev1 finished
Parts:
- added G***: LOGO, Logo:poto, B.Cu at (343.2, 66.5)
- added J15: Power, Connector_PinHeader_1.00mm:PinHeader_1x02_P1.00mm_Vertical, B.Cu at (330.6, 62.2)
- added J16: Power-R, Connector_PinHeader_1.00mm:PinHeader_1x03_P1.00mm_Vertical, B.Cu at (313.1, 71.5)
- added REF**: MountingHole_3.2mm_M3_DIN965_Pad, MountingHole:MountingHole_3.2mm_M3_DIN965_Pad, F.Cu at (60.3, 107.2)
- added REF**: MountingHole_3.2mm_M3_DIN965_Pad, MountingHole:MountingHole_3.2mm_M3_DIN965_Pad, F.Cu at (60.3, 183.4)
- added REF**: MountingHole_3.2mm_M3_DIN965_Pad, MountingHole:MountingHole_3.2mm_M3_DIN965_Pad, F.Cu at (155.6, 183.4)
- added REF**: MountingHole_3.2mm_M3_DIN965_Pad, MountingHole:MountingHole_3.2mm_M3_DIN965_Pad, F.Cu at (155.6, 145.3)
- added REF**: MountingHole_3.2mm_M3_DIN965_Pad, MountingHole:MountingHole_3.2mm_M3_DIN965_Pad, F.Cu at (269.9, 107.2)
- added REF**: MountingHole_3.2mm_M3_DIN965_Pad, MountingHole:MountingHole_3.2mm_M3_DIN965_Pad, F.Cu at (269.9, 183.4)
- added REF**: MountingHole_3.2mm_M3_DIN965_Pad, MountingHole:MountingHole_3.2mm_M3_DIN965_Pad, F.Cu at (269.9, 145.3)
- added REF**: MountingHole_3.2mm_M3_DIN965_Pad, MountingHole:MountingHole_3.2mm_M3_DIN965_Pad, F.Cu at (346.1, 145.3)
- added REF**: MountingHole_3.2mm_M3_DIN965_Pad, MountingHole:MountingHole_3.2mm_M3_DIN965_Pad, F.Cu at (346.1, 183.4)
- added REF**: MountingHole_3.2mm_M3_DIN965_Pad, MountingHole:MountingHole_3.2mm_M3_DIN965_Pad, F.Cu at (346.1, 107.2)
- added REF**: MountingHole_3.2mm_M3_DIN965_Pad, MountingHole:MountingHole_3.2mm_M3_DIN965_Pad, F.Cu at (155.6, 107.2)
- added REF**: MountingHole_3.2mm_M3_DIN965_Pad, MountingHole:MountingHole_3.2mm_M3_DIN965_Pad, F.Cu at (193.7, 183.4)
- added REF**: MountingHole_3.2mm_M3_DIN965_Pad, MountingHole:MountingHole_3.2mm_M3_DIN965_Pad, F.Cu at (193.7, 145.3)
- added REF**: MountingHole_3.2mm_M3_DIN965_Pad, MountingHole:MountingHole_3.2mm_M3_DIN965_Pad, F.Cu at (193.7, 107.2)
- added REF**: MountingHole_3.2mm_M3_DIN965_Pad, MountingHole:MountingHole_3.2mm_M3_DIN965_Pad, F.Cu at (308.0, 183.4)
- added REF**: MountingHole_3.2mm_M3_DIN965_Pad, MountingHole:MountingHole_3.2mm_M3_DIN965_Pad, F.Cu at (308.0, 145.3)
- added REF**: MountingHole_3.2mm_M3_DIN965_Pad, MountingHole:MountingHole_3.2mm_M3_DIN965_Pad, F.Cu at (308.0, 107.2)
- added REF**: MountingHole_3.2mm_M3_DIN965_Pad, MountingHole:MountingHole_3.2mm_M3_DIN965_Pad, F.Cu at (60.3, 145.3)
- SW1: footprint SamacSys_Parts:CMI126601D03 -> keyboard-pcb:2Pin_microswitch
- moved SW1 2.92 mm to (315.8, 66.4), turned to 90 degrees
- moved D1 0.14 mm to (59.2, 101.6)
Routing:
- net +5V: track 141.0 -> 156.5 mm
- net GND: track 206.2 -> 193.9 mm, vias 74 -> 75
- net COL16: track 129.5 -> 136.1 mm
- net /RESET: track 45.8 -> 52.2 mm
- net Net-(D100-Pad2): track 5.06 -> 8.36 mm
- net Net-(D99-Pad2): track 5.08 -> 8.39 mm
- net Net-(D95-Pad2): track 4.91 -> 8.22 mm
- net Net-(D101-Pad2): track 4.99 -> 8.29 mm
- net ROW3: track 440.6 -> 442.0 mm
- net COL6: track 289.4 -> 288.3 mm
- net COL5: track 308.0 -> 307.1 mm
- net COL4: track 326.7 -> 325.9 mm
- net ROW0: track 354.5 -> 355.2 mm
- net COL3: track 347.0 -> 346.4 mm
Other:
- board text added: "5V GND"
